File: XIAO-SX1276.kicad_pcb (KiCad board)
At the start: 2 copper layers, 17.8 x 26.5 mm, 60 parts, among them J1 Conn_01x07, J2 Conn_01x07, J3 Conn_Coaxial_Small, J4 Conn_Coaxial_Small, U1 SX1276, U2 BGS12WN6E6327, U3 BGS12WN6E6327, Y1 32MHz

Commit message: Updates
Parts:
- removed C28: C_Small, Capacitor_SMD:C_0201_0603Metric
- added C24: 100pF, Capacitor_SMD:C_0201_0603Metric, F.Cu at (149.7, 105.1)
- added C25: 100pF, Capacitor_SMD:C_0201_0603Metric, F.Cu at (141.2, 105.1)
- added L11: 15nH, Inductor_SMD:L_0201_0603Metric, F.Cu at (143.6, 112.4)
- C1, C2: value C_Small -> 15pF
- C10: value C_Small -> 8.2pF
- C11, C30, C32: value C_Small -> 6.8pF
- C12, C14, C15, C16, C33, C34, C37: value C_Small -> DNP
- C13, C17: value C_Small -> 3.3pF
- C18, C19, C36, C38, C7, C8: value C_Small -> 47pF
- C29: value C_Small -> 4.7pF
- C31: value C_Small -> 2.7pF
- C35: value C_Small -> 10nF
- C9: value C_Small -> 22pF
- L1: value L_Small -> 82nH
- L10: value L_Small -> 47pF
- L12: value L_Small -> 4.7pF
- L13: value L_Small -> 18nH
- L2: value L_Small -> 33nH
- L3: value L_Small -> 1.5nH
- L4, L5: value L_Small -> 5.6nH
- L6, L8: value L_Small -> 0R
- L7: value L_Small -> 10nH
- L9: value L_Small -> 12nH
- U1: footprint Package_DFN_QFN:QFN-28-1EP_6x6mm_P0.65mm_EP4.8x4.8mm -> Package_DFN_QFN:QFN-28-1EP_6x6mm_P0.65mm_EP4.8x4.8mm_ThermalVias
- Z2, Z5: value TBD -> 0R
- moved C3 0.44 mm to (142.1, 115.5)
- moved C5 0.38 mm to (143.6, 104.7), turned to 90 degrees
- moved J4 0.12 mm to (144.0, 99.0)
- moved J3 0.09 mm to (150.0, 99.0)
Connections:
- C10 pad 1: Net-(U1-VR_PA) -> Net-(C10-Pad1)
- C9 pad 1: Net-(U1-VR_PA) -> Net-(C10-Pad1)
- J1 pad 7: +5V -> unconnected-(J1-Pin_7-Pad7)
- J2 pad 1: /D0 -> unconnected-(J2-Pin_1-Pad1)
- J2 pad 2: /D1 -> unconnected-(J2-Pin_2-Pad2)
- J2 pad 7: /D6/TX -> unconnected-(J2-Pin_7-Pad7)
- L2 pad 1: Net-(L2-Pad1) -> Net-(C10-Pad1)
- L3 pad 2: Net-(L2-Pad1) -> Net-(C10-Pad1)
- U1 pad 16: unconnected-(U1-SCK-Pad16) -> /D8/SCK
- U1 pad 17: unconnected-(U1-MISO-Pad17) -> /D9/MISO
- U1 pad 18: unconnected-(U1-MOSI-Pad18) -> /D10/MOSI
- U1 pad 19: unconnected-(U1-NSS-Pad19) -> /D7/RX
- U1 pad 7: unconnected-(U1-~{RESET}-Pad7) -> /D4/SDA
- U1 pad 8: unconnected-(U1-DIO0-Pad8) -> /D3
- U1 pad 9: unconnected-(U1-DIO1-Pad9) -> /D5/SCL
- U2 pad 6: unconnected-(U2-CTRL-Pad6) -> /D2
- U3 pad 6: unconnected-(U3-CTRL-Pad6) -> /D2
Routing:
- net +3.3V: track 0.00 -> 46.3 mm, vias 0 -> 5
- net GND: track 3.26 -> 30.7 mm, vias 0 -> 63
- net /D3: track 0.00 -> 20.0 mm, vias 0 -> 2
- net /D4/SDA: track 0.00 -> 20.0 mm
- net /D2: track 0.00 -> 18.4 mm, vias 0 -> 2
- net /D5/SCL: track 0.00 -> 17.4 mm, vias 0 -> 1
- net /D10/MOSI: track 0.00 -> 13.0 mm, vias 0 -> 1
- net /D9/MISO: track 0.00 -> 11.8 mm, vias 0 -> 1
- net /D8/SCK: track 0.00 -> 9.78 mm, vias 0 -> 1
- net Net-(U1-VR_PA): track 0.00 -> 7.91 mm, vias 0 -> 2
- net /D7/RX: track 0.00 -> 5.99 mm
- net Net-(U1-XTA): track 0.00 -> 5.32 mm
- net /915MHz_RX: track 0.00 -> 4.38 mm
- net /433MHz_RX: track 0.00 -> 4.37 mm
- net Net-(U1-XTB): track 0.00 -> 3.40 mm
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- added copper zone on B.Cu, net GND
- added copper zone on F.Cu, net GND
- added copper zone on In1.Cu, net GND
- added copper zone on In2.Cu, net GND
Other:
- copper layers 2 -> 4
- board text added: "433MHz"
- board text added: "915MHz"
- board text added: "SX1276"
