File: XIAO-SX1276.kicad_sch (KiCad schematic)
At the start: 60 parts, among them J1 Conn_01x07, J2 Conn_01x07, J3 Conn_Coaxial_Small, J4 Conn_Coaxial_Small, U1 SX1276, U2 BGS12WN6E6327, U3 BGS12WN6E6327, Y1 32MHz

Commit message: Updates
Parts:
- removed C28: C_Small, Capacitor_SMD:C_0201_0603Metric, symbol Device:C_Small
- added C24, C25: 100pF, Capacitor_SMD:C_0201_0603Metric, symbol Device:C_Small
- added L11: 15nH, Inductor_SMD:L_0201_0603Metric, symbol Device:L_Small
- C1, C2: value C_Small -> 10pF; LCSC (none) -> C76921
- C10: value C_Small -> 8.2pF; LCSC (none) -> C85918
- C11, C30, C32: value C_Small -> 6.8pF; LCSC (none) -> C338045
- C12, C14, C15, C16, C33, C34, C37: value C_Small -> DNP; now not fitted; now left out of the parts list
- C13, C17: value C_Small -> 3.3pF; LCSC (none) -> C85906
- C18, C19, C36, C38, C7, C8: value C_Small -> 47pF; LCSC (none) -> C85908
- C20, C21, C22, C23, C3, C4, C5, C6: LCSC (none) -> C76935
- C29: value C_Small -> 4.7pF; LCSC (none) -> C161428
- C31: value C_Small -> 2.7pF; LCSC (none) -> C85902
- C35: value C_Small -> 10nF; LCSC (none) -> C85930
- C9: value C_Small -> 22pF; LCSC (none) -> C76924
- J3, J4: LCSC (none) -> C88374
- L1: value L_Small -> 82nH; LCSC (none) -> C1857896
- L10: value L_Small -> 47pF; LCSC (none) -> C85908
- L12: value L_Small -> 4.7pF; LCSC (none) -> C161428
- L13: value L_Small -> 18nH; LCSC (none) -> C162600
- L2: value L_Small -> 33nH; LCSC (none) -> C162611
- L3: value L_Small -> 1.5nH; LCSC (none) -> C77114
- L4, L5: value L_Small -> 5.6nH; LCSC (none) -> C237444
- L6, L8: value L_Small -> 0R; LCSC (none) -> C22458608
- L7: value L_Small -> 10nH; LCSC (none) -> C162594
- L9: value L_Small -> 12nH; LCSC (none) -> C162597
- U1: footprint Package_DFN_QFN:QFN-28-1EP_6x6mm_P0.65mm_EP4.8x4.8mm -> Package_DFN_QFN:QFN-28-1EP_6x6mm_P0.65mm_EP4.8x4.8mm_ThermalVias; LCSC (none) -> C80171
- U2, U3: LCSC (none) -> C1854968
- Y1: LCSC (none) -> C19858538
- Z1, Z3, Z4, Z6: now not fitted; now left out of the parts list
- Z2, Z5: value TBD -> 0R; LCSC (none) -> C22458608
Connections:
- net D10/MOSI: now also U1.18 (MOSI)
- net D2: now also U2.6 (CTRL), U3.6 (CTRL), C24.2, C25.2
- net D3: now also U1.8 (DIO0)
- net D4/SDA: now also U1.7 (~{RESET})
- net D5/SCL: now also U1.9 (DIO1)
- net D7/RX: now also U1.19 (NSS)
- net D8/SCK: now also U1.16 (SCK)
- net D9/MISO: now also U1.17 (MISO)
- net GND: now also C24.1, C25.1
- net at C29.1, L1.2, U1.28 (RFO_LF): now also L11.1
- net at L8.1: now also L11.2
- net at C35.1, C7.1, C8.1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: no longer C10.1, C9.1
- net at L2.1, L3.2: now also C10.1, C9.1
- net +5V: no longer names the net of J1.7 (Pin_7)
- net D0: no longer names the net of J2.1 (Pin_1)
- net D1: no longer names the net of J2.2 (Pin_2)
- net D6/TX: no longer names the net of J2.7 (Pin_7)
- no-connect marks 1 -> 10
Other:
- moved on the sheet: C1, C10, C11, C13, C17, C18, C19, C2, C20, C21, C22, C23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

Commit message: Updated BOM
Parts:
- U2, U3: LCSC C1854968 -> C285542
Changed lines of the file:
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@@
 			)
 		)
-		(property "LCSC" "C1854968"
+		(property "LCSC" "C285542"
 			(at 0 0 0)
 			(hide yes)
@@
 			)
 		)
-		(property "LCSC" "C1854968"
+		(property "LCSC" "C285542"
 			(at 0 0 0)
 			(hide yes)
